Commit message: Fix mesh path and add missing data files

File: assets/h1_2/h1_2_ros.urdf (robot description, URDF)
Before this commit: robot h1_2, 60 links, 59 joints
Links:
- link L_hand_base_link: geometry collision mesh filename=package://h12_ros2_model/assets/h1_2/meshes/L_hand_base_lin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; visual mesh filename=package://h12_ros2_model/assets/h1_2/meshes/L_hand_base_lin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
- link L_index_intermediate: geometry collision mesh filename=package://h12_ros2_model/assets/h1_2/meshes/link16_L.STL; visual mesh filename=package://h12_ros2_model/assets/h1_2/meshes/link16_L.STL
- link L_index_proximal: geometry collision mesh filename=package://h12_ros2_model/assets/h1_2/meshes/link15_L.STL; visual mesh filename=package://h12_ros2_model/assets/h1_2/meshes/link15_L.STL
- link L_middle_intermediate: geometry collision mesh filename=package://h12_ros2_model/assets/h1_2/meshes/link18_L.STL; visual mesh filename=package://h12_ros2_model/assets/h1_2/meshes/link18_L.STL
- link L_middle_proximal: geometry collision mesh filename=package://h12_ros2_model/assets/h1_2/meshes/link17_L.STL; visual mesh filename=package://h12_ros2_model/assets/h1_2/meshes/link17_L.STL
- link L_pinky_intermediate: geometry collision mesh filename=package://h12_ros2_model/assets/h1_2/meshes/link22_L.STL; visual mesh filename=package://h12_ros2_model/assets/h1_2/meshes/link22_L.STL
- link L_pinky_proximal: geometry collision mesh filename=package://h12_ros2_model/assets/h1_2/meshes/link21_L.STL; visual mesh filename=package://h12_ros2_model/assets/h1_2/meshes/link21_L.STL
- link L_ring_intermediate: geometry collision mesh filename=package://h12_ros2_model/assets/h1_2/meshes/link20_L.STL; visual mesh filename=package://h12_ros2_model/assets/h1_2/meshes/link20_L.STL
- link L_ring_proximal: geometry collision mesh filename=package://h12_ros2_model/assets/h1_2/meshes/link19_L.STL; visual mesh filename=package://h12_ros2_model/assets/h1_2/meshes/link19_L.STL
- link L_thumb_distal: geometry collision mesh filename=package://h12_ros2_model/assets/h1_2/meshes/link14_L.STL; visual mesh filename=package://h12_ros2_model/assets/h1_2/meshes/link14_L.STL
- link L_thumb_intermediate: geometry collision mesh filename=package://h12_ros2_model/assets/h1_2/meshes/link13_L.STL; visual mesh filename=package://h12_ros2_model/assets/h1_2/meshes/link13_L.STL
- link L_thumb_proximal: geometry collision mesh filename=package://h12_ros2_model/assets/h1_2/meshes/link12_L.STL; visual mesh filename=package://h12_ros2_model/assets/h1_2/meshes/link12_L.STL
- link L_thumb_proximal_base: geometry collision mesh filename=package://h12_ros2_model/assets/h1_2/meshes/link11_L.STL; visual mesh filename=package://h12_ros2_model/assets/h1_2/meshes/link11_L.STL
- link R_hand_base_link: geometry collision mesh filename=package://h12_ros2_model/assets/h1_2/meshes/R_hand_base_lin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; visual mesh filename=package://h12_ros2_model/assets/h1_2/meshes/R_hand_base_lin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
- link R_index_intermediate: geometry collision mesh filename=package://h12_ros2_model/assets/h1_2/meshes/link16_R.STL; visual mesh filename=package://h12_ros2_model/assets/h1_2/meshes/link16_R.STL
- link R_index_proximal: geometry collision mesh filename=package://h12_ros2_model/assets/h1_2/meshes/link15_R.STL; visual mesh filename=package://h12_ros2_model/assets/h1_2/meshes/link15_R.STL
- link R_middle_intermediate: geometry collision mesh filename=package://h12_ros2_model/assets/h1_2/meshes/link18_R.STL; visual mesh filename=package://h12_ros2_model/assets/h1_2/meshes/link18_R.STL
- link R_middle_proximal: geometry collision mesh filename=package://h12_ros2_model/assets/h1_2/meshes/link17_R.STL; visual mesh filename=package://h12_ros2_model/assets/h1_2/meshes/link17_R.STL
- link R_pinky_intermediate: geometry collision mesh filename=package://h12_ros2_model/assets/h1_2/meshes/link22_R.STL; visual mesh filename=package://h12_ros2_model/assets/h1_2/meshes/link22_R.STL
- link R_pinky_proximal: geometry collision mesh filename=package://h12_ros2_model/assets/h1_2/meshes/link21_R.STL; visual mesh filename=package://h12_ros2_model/assets/h1_2/meshes/link21_R.STL
- link R_ring_intermediate: geometry collision mesh filename=package://h12_ros2_model/assets/h1_2/meshes/link20_R.STL; visual mesh filename=package://h12_ros2_model/assets/h1_2/meshes/link20_R.STL
- link R_ring_proximal: geometry collision mesh filename=package://h12_ros2_model/assets/h1_2/meshes/link19_R.STL; visual mesh filename=package://h12_ros2_model/assets/h1_2/meshes/link19_R.STL
- link R_thumb_distal: geometry collision mesh filename=package://h12_ros2_model/assets/h1_2/meshes/link14_R.STL; visual mesh filename=package://h12_ros2_model/assets/h1_2/meshes/link14_R.STL
- link R_thumb_intermediate: geometry collision mesh filename=package://h12_ros2_model/assets/h1_2/meshes/link13_R.STL; visual mesh filename=package://h12_ros2_model/assets/h1_2/meshes/link13_R.STL
- link R_thumb_proximal: geometry collision mesh filename=package://h12_ros2_model/assets/h1_2/meshes/link12_R.STL; visual mesh filename=package://h12_ros2_model/assets/h1_2/meshes/link12_R.STL
- link R_thumb_proximal_base: geometry collision mesh filename=package://h12_ros2_model/assets/h1_2/meshes/link11_R.STL; visual mesh filename=package://h12_ros2_model/assets/h1_2/meshes/link11_R.STL
- link left_ankle_pitch_link: geometry collision mesh filename=package://h12_ros2_model/assets/h1_2/meshes/left_ankle_pitc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; visual mesh filename=package://h12_ros2_model/assets/h1_2/meshes/left_ankle_pitc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
- link left_ankle_roll_link: geometry collision mesh filename=package://h12_ros2_model/assets/h1_2/meshes/left_ankle_roll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; visual mesh filename=package://h12_ros2_model/assets/h1_2/meshes/left_ankle_roll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
- link left_elbow_pitch_link: geometry collision mesh filename=package://h12_ros2_model/assets/h1_2/meshes/left_elbow_pitc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; visual mesh filename=package://h12_ros2_model/assets/h1_2/meshes/left_elbow_pitc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
- link left_elbow_roll_link: geometry collision mesh filename=package://h12_ros2_model/assets/h1_2/meshes/left_elbow_roll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; visual mesh filename=package://h12_ros2_model/assets/h1_2/meshes/left_elbow_roll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
- link left_hip_pitch_link: geometry collision cylinder length=0.2 radius=0.02; visual mesh filename=package://h12_ros2_model/assets/h1_2/meshes/left_hip_pitch_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
- link left_hip_roll_link: geometry collision cylinder length=0.01 radius=0.02; visual mesh filename=package://h12_ros2_model/assets/h1_2/meshes/left_hip_roll_l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
- link left_hip_yaw_link: geometry collision cylinder length=0.02 radius=0.01; visual mesh filename=package://h12_ros2_model/assets/h1_2/meshes/left_hip_yaw_li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
- link left_knee_link: geometry collision cylinder length=0.2 radius=0.02; visual mesh filename=package://h12_ros2_model/assets/h1_2/meshes/left_knee_link.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
- link left_shoulder_pitch_link: geometry collision mesh filename=package://h12_ros2_model/assets/h1_2/meshes/left_shoulder_p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; visual mesh filename=package://h12_ros2_model/assets/h1_2/meshes/left_shoulder_p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
- link left_shoulder_roll_link: geometry collision mesh filename=package://h12_ros2_model/assets/h1_2/meshes/left_shoulder_r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; visual mesh filename=package://h12_ros2_model/assets/h1_2/meshes/left_shoulder_r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
- link left_shoulder_yaw_link: geometry collision mesh filename=package://h12_ros2_model/assets/h1_2/meshes/left_shoulder_y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; visual mesh filename=package://h12_ros2_model/assets/h1_2/meshes/left_shoulder_y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
- link left_wrist_pitch_link: geometry collision mesh filename=package://h12_ros2_model/assets/h1_2/meshes/left_wrist_pitc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; visual mesh filename=package://h12_ros2_model/assets/h1_2/meshes/left_wrist_pitc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
- link left_wrist_yaw_link: geometry visual mesh filename=package://h12_ros2_model/assets/h1_2/meshes/wrist_yaw_link.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
- link logo_link: geometry visual mesh filename=package://h12_ros2_model/assets/h1_2/meshes/logo_link.STL
- link pelvis: geometry collision sphere radius=0.05; visual mesh filename=package://h12_ros2_model/assets/h1_2/meshes/pelvis.STL
- link right_ankle_pitch_link: geometry collision mesh filename=package://h12_ros2_model/assets/h1_2/meshes/right_ankle_pit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; visual mesh filename=package://h12_ros2_model/assets/h1_2/meshes/right_ankle_pit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
- link right_ankle_roll_link: geometry collision mesh filename=package://h12_ros2_model/assets/h1_2/meshes/right_ankle_rol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; visual mesh filename=package://h12_ros2_model/assets/h1_2/meshes/right_ankle_rol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
- link right_elbow_pitch_link: geometry collision mesh filename=package://h12_ros2_model/assets/h1_2/meshes/right_elbow_pit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; visual mesh filename=package://h12_ros2_model/assets/h1_2/meshes/right_elbow_pit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
- link right_elbow_roll_link: geometry collision mesh filename=package://h12_ros2_model/assets/h1_2/meshes/right_elbow_rol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; visual mesh filename=package://h12_ros2_model/assets/h1_2/meshes/right_elbow_rol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
- link right_hip_pitch_link: geometry collision cylinder length=0.2 radius=0.02; visual mesh filename=package://h12_ros2_model/assets/h1_2/meshes/right_hip_pitch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
- link right_hip_roll_link: geometry collision cylinder length=0.01 radius=0.02; visual mesh filename=package://h12_ros2_model/assets/h1_2/meshes/right_hip_roll_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
- link right_hip_yaw_link: geometry collision cylinder length=0.02 radius=0.01; visual mesh filename=package://h12_ros2_model/assets/h1_2/meshes/right_hip_yaw_l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
- link right_knee_link: geometry collision cylinder length=0.2 radius=0.02; visual mesh filename=package://h12_ros2_model/assets/h1_2/meshes/right_knee_link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
- link right_shoulder_pitch_link: geometry collision mesh filename=package://h12_ros2_model/assets/h1_2/meshes/right_shoulder_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; visual mesh filename=package://h12_ros2_model/assets/h1_2/meshes/right_shoulder_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
- link right_shoulder_roll_link: geometry collision mesh filename=package://h12_ros2_model/assets/h1_2/meshes/right_shoulder_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; visual mesh filename=package://h12_ros2_model/assets/h1_2/meshes/right_shoulder_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
- link right_shoulder_yaw_link: geometry collision mesh filename=package://h12_ros2_model/assets/h1_2/meshes/right_shoulder_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; visual mesh filename=package://h12_ros2_model/assets/h1_2/meshes/right_shoulder_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
- link right_wrist_pitch_link: geometry collision mesh filename=package://h12_ros2_model/assets/h1_2/meshes/right_wrist_pit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; visual mesh filename=package://h12_ros2_model/assets/h1_2/meshes/right_wrist_pit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
- link right_wrist_yaw_link: geometry visual mesh filename=package://h12_ros2_model/assets/h1_2/meshes/wrist_yaw_link.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
- link torso_link: geometry collision box size=0.08 0.16 0.1; visual mesh filename=package://h12_ros2_model/assets/h1_2/meshes/torso_link.STL
